File: hardware/logicboard/p2-001.sch (EAGLE design)
At the start: 13 parts, among them IC1 74LS07N, IC5 5V

Commit message: Schematic.
Parts:
- removed IC5: 5V, v-reg:78XXL
- added C4, C5: 103, rcl:C-US025-025X050
- added D2: DIODE-1N4148, SparkFun-DiscreteSemi:DIODE-1N4148
- added IC2: 74LS07N, 74xx-us:74LS07N
- added K1: G5V1, relay:G5V1
- added R1, R2: (no value), resistor:R-EU_0204/5
- added RN2, RN3: (no value), resistor-net:RN08
- added T1: 2SC1815, transistor:2SC1815
- added U1: DS18B20, SparkFun-Sensors:DS18B20
- IC1: value 74LS07N -> 5V; device 74xx-us:74LS07N -> v-reg:78XXL
Connections:
- net MIDIINA renamed MIDIINSND
- removed net +12V: C1.1, IC5.IN, MC1.9V
- removed net N$3: IC1B.O, RN1E.1
- removed net N$4: IC1C.O, RN1G.1
- removed net N$5: IC1A.O, RN1C.1
- removed net N$6: C2.1, IC5.OUT
- new net 12V: K12.O, MC1.9V, SV2-1.S
- new net 12VRLY: C1.1, IC1.IN, K12.P, K12.P@1
- new net A1: MC1.A0, SV1-4.S
- new net A2: MC1.A1, SV1-10.S
- new net A3: MC1.A2, SV1-16.S
- new net A4: MC1.A3, SV1-22.S
- new net CLK: MC1.SCK, SV2-13.S
- new net D1: MC1.6, RN3.4, SV1-3.S
- new net D2: MC1.9, RN3.5, SV1-9.S
- new net D3: MC1.10, RN3.6, SV1-15.S
- new net D4: MC1.12, RN3.7, SV1-21.S
- new net GPIO: MC1.5, SV2-9.S
- new net LED0: MC1.13, SV1-25.S
- new net LED0K: RN2.2, SV1-26.S
- new net LED1: MC1.4, SV1-27.S
- new net LED1K: RN2.3, SV1-28.S
- new net LED2: MC1.7, SV1-29.S
- new net LED2K: RN2.4, SV1-30.S
- new net LED3: MC1.8, SV1-31.S
- new net LED3K: RN2.5, SV1-32.S
- new net LED4: MC1.11, SV1-33.S
- new net LED4K: RN2.6, SV1-34.S
- new net MIDIOUT2RTN: IC2C.O, RN1G.1
- new net MIDIOUTRTN: IC2B.O, RN1E.1
- new net MIDITHRURTN: IC2A.O, RN1C.1
- new net MISO: MC1.MISO, SV2-14.S
- new net MOSI: MC1.MOSI, SV2-12.S
- new net N$10: RN1C.2, SV2-18.S
- new net N$11: RN1F.2, SV2-15.S
- new net N$12: RN1G.2, SV2-16.S
- new net N$2: RN1A.2, SV2-5.S
- new net N$7: RN1D.2, SV2-10.S
- new net N$8: RN1E.2, SV2-11.S
- new net N$9: RN1B.2, SV2-17.S
- new net RLY: MC1.A5, R1.2
- new net RLYDRV: R1.1, R2.2, T1.B
- new net RLYSNK: D2.A, K11.2, T1.C
- new net RST: MC1.R@2, SV2-3.S
- new net SCL: MC1.3, RN3.3, SV1-12.S, SV1-18.S, SV1-24.S, SV1-6.S
- new net SDA: MC1.2, RN3.2, SV1-11.S, SV1-17.S, SV1-23.S, SV1-5.S
- new net THS: MC1.A4, RN3.8, U1.DQ
- new net VDD: MC1.3V, SV2-19.S
- new net VOUT: C2.1, IC1.OUT, SV1-1.S, SV1-13.S, SV1-19.S, SV1-7.S
- net GND: now also C4.2, C5.2, IC1.GND, IC2D.I, IC2E.I, IC2F.I, MC1.GND@1, R2.1, RN2.1, SV1-14.S, SV1-2.S, SV1-20.S, SV1-8.S, SV2-2.S, SV2-20.S, SV2-4.S, SV2-8.S, T1.E, U1.GND; no longer IC5.GND
- net N$1: now also SV2-6.S
- net RX: now also IC2A.I, MC1.RX; no longer IC1A.I
- net TX: now also IC2B.I, IC2C.I, MC1.TX; no longer IC1B.I, IC1C.I
- net VCC: now also C4.1, C5.1, D2.C, K11.1, RN3.1, SV2-7.S, U1.VDD
Other:
- moved on the sheet: C1, C2, C3, D1, OK1, RN1A, RN1B, RN1C, RN1D, RN1E, RN1F, RN1G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

Commit message: Refine of schematic and board.
Other:
- moved on the sheet: C1, C2, C3, C4, C5, D1, D2, IC1, IC2A, IC2B, IC2C, IC2D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

Commit message: Layout.
Parts:
- added JP1: GNDPIN, pinhead:PINHD-1X1
- added RN4: Optional, resistor-net:RN04
- R1: value (none) -> 1k
- R2: value (none) -> 47k
- RN2: value (none) -> 330
- RN3: value (none) -> 4.7k
Connections:
- net 12V renamed +12V
- net A1: now also RN4.2
- net A2: now also RN4.3
- net A3: now also RN4.4
- net A4: now also RN4.5
- net GND: now also JP1.1
- net VCC: now also RN4.1

Commit message: Board design.
Changed lines of the file:
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@@
 <?xml version="1.0" encoding="utf-8"?>
 <!DOCTYPE eagle SYSTEM "eagle.dtd">
-<eagle version="9.4.2">
+<eagle version="9.5.2">
 <drawing>
 <settings>
@@
 <bus name="INTL:RLY,THS">
 <segment>
-<wire x1="223.52" y1="172.72" x2="190.5" y2="172.72" width="0.762" layer="92"/>
-<wire x1="190.5" y1="172.72" x2="187.96" y2="170.18" width="0.762" layer="92" curve="90"/>
-<wire x1="187.96" y1="170.18" x2="187.96" y2="132.08" width="0.762" layer="92"/>
-<wire x1="187.96" y1="132.08" x2="185.42" y2="129.54" width="0.762" layer="92" curve="-90"/>
-<wire x1="185.42" y1="129.54" x2="180.34" y2="129.54" width="0.762" layer="92"/>
-<wire x1="180.34" y1="129.54" x2="177.8" y2="132.08" width="0.762" layer="92" curve="-90"/>
-<wire x1="177.8" y1="132.08" x2="177.8" y2="218.44" width="0.762" layer="92"/>
-<label x="180.34" y="129.54" size="1.778" layer="95"/>
+<wire x1="223.52" y1="172.72" x2="180.34" y2="172.72" width="0.762" layer="92"/>
+<wire x1="180.34" y1="172.72" x2="177.8" y2="175.26" width="0.762" layer="92" curve="-90"/>
+<wire x1="177.8" y1="175.26" x2="177.8" y2="218.44" width="0.762" layer="92"/>
+<label x="180.34" y="172.72" size="1.778" layer="95"/>
 </segment>
 </bus>

Commit message: XLED terminals.
Parts:
- added C6: 103, rcl:C-US025-025X050
- added IC3: 4066N, 40xx:4066N
- added JP2: (no value), pinhead:PINHD-1X2
- RN4: value Optional -> 10k
Connections:
- removed net CLK: MC1.SCK, SV2-13.S
- removed net GPIO: MC1.5, SV2-9.S
- removed net MOSI: MC1.MOSI, SV2-12.S
- new net N$13: IC2D.O, SV2-12.S
- new net N$14: IC2E.O, SV2-13.S
- new net N$15: IC2F.O, SV2-14.S
- new net N$3: IC3A.A, RN4.2
- new net N$4: IC3B.A, RN4.3
- new net N$5: IC3C.A, RN4.4
- new net N$6: IC3D.A, RN4.5
- new net PULLUP: IC3A.C, IC3B.C, IC3C.C, IC3D.C, MC1.7
- net +12V: now also JP2.1
- net 12VRLY: now also JP2.2
- net A1: now also IC3A.B; no longer RN4.2
- net A2: now also IC3B.B; no longer RN4.3
- net A3: now also IC3C.B; no longer RN4.4
- net A4: now also IC3D.B; no longer RN4.5
- net GND: now also C6.2; no longer IC2D.I, IC2E.I, IC2F.I
- net LED0: now also IC2D.I
- net LED2: now also IC2E.I, MC1.5; no longer MC1.7
- net LED4: now also IC2F.I
- net MISO: no longer SV2-14.S
- net RST: now also MC1.R@1; no longer MC1.R@2
- net THS: now also SV2-9.S
- net VCC: now also C6.1
Other:
- moved on the sheet: C1, C3, C4, C5, D1, D2, IC2A, IC2B, IC2C, IC2D, IC2E, IC2F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

Commit message: Clean up.
Connections:
- net N$1 renamed MINRTN
- net N$10 renamed MTHRTN
- net N$11 renamed MO2SND
- net N$12 renamed MO2RTN
- net N$13 renamed XLEDG
- net N$14 renamed XLEDB
- net N$15 renamed XLEDR
- net N$2 renamed MINSND
- net N$7 renamed MO1SND
- net N$8 renamed MO1RTN
- net N$9 renamed MTHSND
- removed net MISO: MC1.MISO
- net GND: now also IC3P.VSS
- net VCC: now also IC3P.VDD
Other:
- moved on the sheet: C1, C2, C3, C4, C5, C6, D1, D2, IC1, IC2A, IC2B, IC2C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
